File: renders/Tic_Tac_Toe_2.0.brd (EAGLE design)
At the start: 55.9 x 53 mm, 44 parts, among them J1 C10418, Q2 16 MHZ, U1 ATMEGA328PB-AUR, U2 LM7805S/NOPB

Commit message: 2.2
Parts:
- added U$11, U$12, U$13: FIDUCIAL, adafruit:FIDUCIAL_1MM
- H1, H2, H3: value MOUNT-HOLE2.8 -> MOUNT-HOLE3.0; device holes:2,8 -> holes:3,0
- moved H1 44.7 mm to (19.1, 30.5)
- moved C11 4.58 mm to (12.7, 26.7)
- moved H3 2.54 mm to (14.0, 64.8), turned to 180 degrees
- moved PAD2 2.54 mm to (12.7, 31.8)
- moved U$1 2.54 mm to (61.0, 22.9)
- moved C6 1.80 mm to (19.1, 40.6)
- moved C10 1.27 mm to (15.2, 40.6)
- moved C15 1.27 mm to (50.8, 25.4), turned to 180 degrees
- moved PAD1 1.27 mm to (12.7, 35.6)
- moved R1 1.27 mm to (50.8, 27.9), turned to 0 degrees
Routing:
- net VCC: track 250.6 -> 71.6 mm, vias 13 -> 16
- net GND: track 9.03 -> 19.8 mm, vias 1 -> 2
- net MOSI: track 61.7 -> 57.4 mm
- net RST: track 31.2 -> 33.2 mm
- net PD0: track 71.1 -> 73.0 mm
- net SCK: track 48.9 -> 50.3 mm
- net N$4: track 14.0 -> 12.6 mm
- net PD1: track 56.8 -> 55.7 mm
- net MISO: track 14.2 -> 13.1 mm
- added copper zone on layer 16, net VCC
- removed copper zone on layer 16, net GND
Other:
- board text added: "Filipe Raposo Tic-tac-toe Fall 2020 https://github.com/fviveirosraposo"
- board text removed: "Filipe Raposo Tic-tac-toe 11/8/2020 https://github.com/fviveirosraposo"
